Commit message: initial position fixed to aim at the ball

File: ball/sphere_small.urdf (robot description, URDF)
Before this commit: robot urdf_robot, 1 links, 0 joints
Links:
- link base_link: geometry collision sphere radius=0.05; visual mesh filename=textured_sphere_smooth.obj scale=0.05 0.05 0.05
